File: helpers/ignitor_mux.brd (EAGLE design)
At the start: 28 x 24 mm, 4 parts, among them J1 S2B-PH-K-S(LF)(SN), J2 S2B-PH-K-S(LF)(SN), J3 S2B-PH-K-S(LF)(SN), J4 S2B-PH-K-S(LF)(SN)

Commit message: helper boards prod files
Other:
- board text added: "Designed by ART"
- board text added: "JLCJLCJLCJLC"
Changed lines of the file:
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@@
 <layer number="27" name="tValues" color="7" fill="1" visible="no" active="yes"/>
 <layer number="28" name="bValues" color="7" fill="1" visible="no" active="yes"/>
-<layer number="29" name="tStop" color="7" fill="3" visible="no" active="yes"/>
-<layer number="30" name="bStop" color="7" fill="6" visible="no" active="yes"/>
+<layer number="29" name="tStop" color="7" fill="3" visible="yes" active="yes"/>
+<layer number="30" name="bStop" color="7" fill="6" visible="yes" active="yes"/>
 <layer number="31" name="tCream" color="7" fill="4" visible="no" active="yes"/>
 <layer number="32" name="bCream" color="7" fill="5" visible="no" active="yes"/>
@@
 <dimension x1="15" y1="8" x2="15" y2="-9" x3="18" y3="-0.5" textsize="1.778" textratio="15" layer="47"/>
 <dimension x1="6" y1="0" x2="-6" y2="0" x3="0" y3="-3" textsize="1.778" textratio="15" layer="47"/>
-<hole x="-10" y="0" drill="4"/>
+<hole x="-10" y="0" drill="4.2"/>
 <rectangle x1="-0.49" y1="-4.11" x2="0.49" y2="-4.09" layer="30" rot="R180"/>
 <rectangle x1="-0.61" y1="-4.09" x2="0.61" y2="-4.07" layer="30" rot="R180"/>
@@
 <text x="5" y="-1" size="1" layer="22" font="vector" ratio="15" rot="MR270">Ignitor B</text>
 <text x="5" y="7" size="1" layer="22" font="vector" ratio="15" rot="MR270">Ignitor A</text>
-<hole x="0" y="6" drill="3"/>
-<hole x="0" y="-7" drill="3"/>
-<text x="-10" y="9" size="2" layer="21" font="vector" ratio="15">+</text>
-<text x="-10" y="-7" size="2" layer="21" font="vector" ratio="15">+</text>
-<text x="8" y="1" size="2" layer="21" font="vector" ratio="15">+</text>
-<text x="8" y="-7" size="2" layer="21" font="vector" ratio="15">+</text>
-<text x="-10" y="5" size="2" layer="21" font="vector" ratio="15">-</text>
-<text x="-10" y="-11" size="2" layer="21" font="vector" ratio="15">-</text>
-<text x="8" y="-3" size="2" layer="21" font="vector" ratio="15">-</text>
-<text x="8" y="5" size="2" layer="21" font="vector" ratio="15">-</text>
-<text x="-9" y="9" size="2" layer="22" font="vector" ratio="15" rot="MR0">+</text>
-<text x="-9" y="5" size="2" layer="22" font="vector" ratio="15" rot="MR0">-</text>
-<text x="-9" y="-7" size="2" layer="22" font="vector" ratio="15" rot="MR0">+</text>
-<text x="-9" y="-11" size="2" layer="22" font="vector" ratio="15" rot="MR0">-</text>
-<text x="10" y="-7" size="2" layer="22" font="vector" ratio="15" rot="MR0">+</text>
-<text x="10" y="-3" size="2" layer="22" font="vector" ratio="15" rot="MR0">-</text>
-<text x="10" y="1" size="2" layer="22" font="vector" ratio="15" rot="MR0">+</text>
-<text x="10" y="5" size="2" layer="22" font="vector" ratio="15" rot="MR0">-</text>
+<hole x="0" y="5.492" drill="3"/>
+<hole x="0" y="-6.492" drill="3"/>
+<text x="-10.254" y="7.984" size="2" layer="21" font="vector" ratio="15">+</text>
+<text x="-10.254" y="-7.889" size="2" layer="21" font="vector" ratio="15">+</text>
+<text x="8.762" y="2.143" size="2" layer="21" font="vector" ratio="15">+</text>
+<text x="8.762" y="-5.984" size="2" layer="21" font="vector" ratio="15">+</text>
+<text x="-10.127" y="6.016" size="2" layer="21" font="vector" ratio="15">-</text>
+<text x="-10.254" y="-9.857" size="2" layer="21" font="vector" ratio="15">-</text>
+<text x="8.762" y="-3.762" size="2" layer="21" font="vector" ratio="15">-</text>
+<text x="8.762" y="4.238" size="2" layer="21" font="vector" ratio="15">-</text>
+<text x="-8.873" y="7.984" size="2" layer="22" font="vector" ratio="15" rot="MR0">+</text>
+<text x="-8.746" y="6.016" size="2" layer="22" font="vector" ratio="15" rot="MR0">-</text>
+<text x="-8.873" y="-7.889" size="2" layer="22" font="vector" ratio="15" rot="MR0">+</text>
+<text x="-8.873" y="-9.857" size="2" layer="22" font="vector" ratio="15" rot="MR0">-</text>
+<text x="10.254" y="-5.984" size="2" layer="22" font="vector" ratio="15" rot="MR0">+</text>
+<text x="10.254" y="-3.762" size="2" layer="22" font="vector" ratio="15" rot="MR0">-</text>
+<text x="10.254" y="2.143" size="2" layer="22" font="vector" ratio="15" rot="MR0">+</text>
+<text x="10.254" y="4.238" size="2" layer="22" font="vector" ratio="15" rot="MR0">-</text>
 <rectangle x1="-0.49" y1="-4.11" x2="0.49" y2="-4.09" layer="29"/>
 <rectangle x1="-0.61" y1="-4.09" x2="0.61" y2="-4.07" layer="29"/>
@@
 <rectangle x1="-0.51" y1="3.25" x2="0.51" y2="3.27" layer="29"/>
 <rectangle x1="-0.29" y1="3.27" x2="0.29" y2="3.29" layer="29"/>
+<text x="5.842" y="-2.032" size="0.85" layer="21" font="vector" ratio="20">JLCJLCJLCJLC</text>
+<text x="12.7" y="6.35" size="1.2" layer="22" font="vector" ratio="15" rot="MR270">Designed by ART</text>
 </plain>
 <attributes>
@@
 </class>
 </classes>
-<designrules name="default">
-<description language="de">&lt;b&gt;EAGLE Design Rules&lt;/b&gt;
-&lt;p&gt;
-Die Standard-Design-Rules sind so gewählt, dass sie für
-die meisten Anwendungen passen. Sollte ihre Platine
-besondere Anforderungen haben, treffen Sie die erforderlichen
-Einstellungen hier und speichern die Design Rules unter
-einem neuen Namen ab.</description>
-<description language="en">&lt;b&gt;EAGLE Design Rules&lt;/b&gt;
-&lt;p&gt;
-The default Design Rules have been set to cover
-a wide range of applications. Your particular design
-may have different requirements, so please make the
-necessary adjustments and save your customized
-design rules under a new name.</description>
+<designrules name="jlcpcb-2layers">
+<description language="en">&lt;b&gt;JLCPCB design rules (2 layers)&lt;/b&gt;
+&lt;ul&gt;
+&lt;li&gt;Board thickness: 1.6mm&lt;/li&gt;
+&lt;li&gt;Copper weight: 1oz (35um)&lt;/li&gt;
+&lt;li&gt;Note: annular ring aren't minimal&lt;/li&gt;
+&lt;/ul&gt;</description>
 <param name="layerSetup" value="(1*16)"/>
 <param name="mtCopper" value="0.035mm 0.035mm 0.035mm 0.035mm 0.035mm 0.035mm 0.035mm 0.035mm 0.035mm 0.035mm 0.035mm 0.035mm 0.035mm 0.035mm 0.035mm 0.035mm"/>
-<param name="mtIsolate" value="1.5mm 0.15mm 0.2mm 0.15mm 0.2mm 0.15mm 0.2mm 0.15mm 0.2mm 0.15mm 0.2mm 0.15mm 0.2mm 0.15mm 0.2mm"/>
-<param name="mdWireWire" value="6mil"/>
-<param name="mdWirePad" value="6mil"/>
-<param name="mdWireVia" value="6mil"/>
-<param name="mdPadPad" value="6mil"/>
-<param name="mdPadVia" value="6mil"/>
-<param name="mdViaVia" value="6mil"/>
-<param name="mdSmdPad" value="6mil"/>
-<param name="mdSmdVia" value="6mil"/>
-<param name="mdSmdSmd" value="6mil"/>
+<param name="mtIsolate" value="1.6mm 0.15mm 0.2mm 0.15mm 0.2mm 0.15mm 0.2mm 0.15mm 0.2mm 0.15mm 0.2mm 0.15mm 0.2mm 0.15mm 0.2mm"/>
+<param name="mdWireWire" value="5mil"/>
+<param name="mdWirePad" value="5mil"/>
+<param name="mdWireVia" value="5mil"/>
+<param name="mdPadPad" value="5mil"/>
+<param name="mdPadVia" value="5mil"/>
+<param name="mdViaVia" value="5mil"/>
+<param name="mdSmdPad" value="5mil"/>
+<param name="mdSmdVia" value="5mil"/>
+<param name="mdSmdSmd" value="5mil"/>
 <param name="mdViaViaSameLayer" value="6mil"/>
 <param name="mnLayersViaInSmd" value="2"/>
-<param name="mdCopperDimension" value="40mil"/>
+<param name="mdCopperDimension" value="0.2mm"/>
 <param name="mdDrill" value="6mil"/>
 <param name="mdSmdStop" value="0mil"/>
-<param name="msWidth" value="6mil"/>
-<param name="msDrill" value="0.35mm"/>
-<param name="msMicroVia" value="9.99mm"/>
+<param name="msWidth" value="5mil"/>
+<param name="msDrill" value="0.3mm"/>
+<param name="msMicroVia" value="0.3mm"/>
 <param name="msBlindViaRatio" value="0.5"/>
-<param name="rvPadTop" value="0.25"/>
-<param name="rvPadInner" value="0.25"/>
-<param name="rvPadBottom" value="0.25"/>
-<param name="rvViaOuter" value="0.25"/>
-<param name="rvViaInner" value="0.25"/>
-<param name="rvMicroViaOuter" value="0.25"/>
-<param name="rvMicroViaInner" value="0.25"/>
+<param name="rvPadTop" value="0.4"/>
+<param name="rvPadInner" value="0"/>
+<param name="rvPadBottom" value="0.4"/>
+<param name="rvViaOuter" value="0"/>
+<param name="rvViaInner" value="0"/>
+<param name="rvMicroViaOuter" value="0"/>
+<param name="rvMicroViaInner" value="0"/>
 <param name="rlMinPadTop" value="10mil"/>
-<param name="rlMaxPadTop" value="20mil"/>
+<param name="rlMaxPadTop" value="80mil"/>
 <param name="rlMinPadInner" value="10mil"/>
 <param name="rlMaxPadInner" value="20mil"/>
 <param name="rlMinPadBottom" value="10mil"/>
-<param name="rlMaxPadBottom" value="20mil"/>
-<param name="rlMinViaOuter" value="8mil"/>
+<param name="rlMaxPadBottom" value="80mil"/>
+<param name="rlMinViaOuter" value="3mil"/>
 <param name="rlMaxViaOuter" value="20mil"/>
 <param name="rlMinViaInner" value="8mil"/>
 <param name="rlMaxViaInner" value="20mil"/>
-<param name="rlMinMicroViaOuter" value="4mil"/>
+<param name="rlMinMicroViaOuter" value="3mil"/>
 <param name="rlMaxMicroViaOuter" value="20mil"/>
 <param name="rlMinMicroViaInner" value="4mil"/>
