File: helpers/jst_splitter.brd (EAGLE design)
At the start: 19.8 x 14.3 mm, 3 parts, among them J1 S2B-PH-K-S(LF)(SN), J2 S2B-PH-K-S(LF)(SN), J3 S2B-PH-K-S(LF)(SN)

Commit message: helper boards prod files
Connections:
- removed net FIRE: J1.1, J3.1
- new net VCC: J1.2, J2.2, J3.2
- net GND: now also J1.1, J2.1, J3.1; no longer J1.2, J3.2
Routing:
- added copper zone on layer 1, net VCC
- removed copper zone on layer 1, net FIRE
Other:
- board text removed: "JLCJLCJLCJLC"
Changed lines of the file:
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@@
 <layer number="48" name="Document" color="7" fill="1" visible="no" active="yes"/>
 <layer number="49" name="Reference" color="7" fill="1" visible="no" active="yes"/>
-<layer number="51" name="tDocu" color="6" fill="1" visible="yes" active="yes"/>
+<layer number="51" name="tDocu" color="6" fill="1" visible="no" active="yes"/>
 <layer number="52" name="bDocu" color="7" fill="1" visible="no" active="yes"/>
 <layer number="88" name="SimResults" color="9" fill="1" visible="no" active="no"/>
@@
 <text x="6.7" y="-6.1" size="2.5" layer="22" font="vector" ratio="12" rot="MR90">OUT</text>
 <text x="6.8" y="1.6" size="2.5" layer="22" font="vector" ratio="12" rot="MR90">OUT</text>
-<text x="-5.5" y="1.1" size="2.5" layer="21" font="vector" ratio="12">+</text>
-<text x="4" y="-6.3" size="2.5" layer="21" font="vector" ratio="12">+</text>
-<text x="4" y="1.5" size="2.5" layer="21" font="vector" ratio="12">+</text>
-<text x="-5.5" y="-3.3" size="2.5" layer="21" font="vector" ratio="12">-</text>
-<text x="4.1" y="-2.1" size="2.5" layer="21" font="vector" ratio="12">-</text>
-<text x="4.1" y="5.5" size="2.5" layer="21" font="vector" ratio="12">-</text>
-<text x="-3.7" y="1.1" size="2.5" layer="22" font="vector" ratio="12" rot="MR0">+</text>
-<text x="-3.7" y="-3.3" size="2.5" layer="22" font="vector" ratio="12" rot="MR0">-</text>
-<text x="5.8" y="-6.3" size="2.5" layer="22" font="vector" ratio="12" rot="MR0">+</text>
-<text x="5.9" y="-2.1" size="2.5" layer="22" font="vector" ratio="12" rot="MR0">-</text>
-<text x="5.8" y="1.5" size="2.5" layer="22" font="vector" ratio="12" rot="MR0">+</text>
-<text x="5.9" y="5.5" size="2.5" layer="22" font="vector" ratio="12" rot="MR0">-</text>
-<text x="-1.7" y="-2.5" size="0.5" layer="21" rot="R90">JLCJLCJLCJLC</text>
+<text x="-6.1" y="-2" size="2.5" layer="21" font="vector" ratio="12">+</text>
+<text x="4.3" y="-3.3" size="2.5" layer="21" font="vector" ratio="12">+</text>
+<text x="4.3" y="4.4" size="2.5" layer="21" font="vector" ratio="12">+</text>
+<text x="-6.1" y="0" size="2.5" layer="21" font="vector" ratio="12">-</text>
+<text x="4.3" y="-5.3" size="2.5" layer="21" font="vector" ratio="12">-</text>
+<text x="4.3" y="2.4" size="2.5" layer="21" font="vector" ratio="12">-</text>
+<text x="-4.3" y="-2" size="2.5" layer="22" font="vector" ratio="12" rot="MR0">+</text>
+<text x="-4.3" y="0" size="2.5" layer="22" font="vector" ratio="12" rot="MR0">-</text>
+<text x="6.1" y="-3.3" size="2.5" layer="22" font="vector" ratio="12" rot="MR0">+</text>
+<text x="6.1" y="-5.3" size="2.5" layer="22" font="vector" ratio="12" rot="MR0">-</text>
+<text x="6.1" y="4.4" size="2.5" layer="22" font="vector" ratio="12" rot="MR0">+</text>
+<text x="6.1" y="2.4" size="2.5" layer="22" font="vector" ratio="12" rot="MR0">-</text>
 </plain>
 <attributes>
@@
 </elements>
 <signals>
-<signal name="FIRE">
+<signal name="GND">
+<polygon width="0.2" layer="16" spacing="0.15">
+<vertex x="-13.2" y="11"/>
+<vertex x="13.2" y="11"/>
+<vertex x="13.2" y="-9.9"/>
+<vertex x="-13.2" y="-9.9"/>
+</polygon>
+<contactref element="J3" pad="1"/>
 <contactref element="J1" pad="1"/>
-<contactref element="J3" pad="1"/>
+<contactref element="J2" pad="1"/>
+</signal>
+<signal name="VCC">
+<contactref element="J3" pad="2"/>
+<contactref element="J1" pad="2"/>
+<contactref element="J2" pad="2"/>
 <polygon width="0.2" layer="1" spacing="0.15">
 <vertex x="-11" y="8.8"/>
@@
 </polygon>
 </signal>
-<signal name="GND">
-<contactref element="J3" pad="2"/>
-<contactref element="J1" pad="2"/>
-<polygon width="0.2" layer="16" spacing="0.15">
-<vertex x="-13.2" y="11"/>
-<vertex x="13.2" y="11"/>
-<vertex x="13.2" y="-9.9"/>
-<vertex x="-13.2" y="-9.9"/>
-</polygon>
-</signal>
